File: OtterX_RamExp.kicad_sch (KiCad schematic)
At the start: 9 parts, among them J1 RAM Exp Connector, U1 AS6C4008-55PCN, U2 AS6C4008-55PCN, U3 AS6C4008-55PCN, U4 74ACT139

Commit message: Update the PCB
Parts:
- U4: value 74ACT139 -> 74AC139
Changed lines of the file:
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@@
 			)
 		)
-		(property "Value" "74ACT139"
+		(property "Value" "74AC139"
 			(at 142.24 120.65 0)
 			(effects
@@
 			)
 		)
-		(property "Value" "74ACT139"
+		(property "Value" "74AC139"
 			(at 64.77 119.38 0)
 			(effects
@@
 			)
 		)
-		(property "Value" "74ACT139"
+		(property "Value" "74AC139"
 			(at 248.92 133.3499 0)
 			(effects
