File: OtterX_RamExp.kicad_pcb (KiCad board)
At the start: 2 copper layers, 52.8 x 40.4 mm, 9 parts, among them J1 RAM Exp Connector, U1 AS6C4008-55PCN, U2 AS6C4008-55PCN, U3 AS6C4008-55PCN, U4 74ACT139

Commit message: Update the PCB
Parts:
- U4: value 74ACT139 -> 74AC139
Routing:
- net GND: track 207.6 -> 209.9 mm, vias 5 -> 8
Changed lines of the file:
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@@
 			)
 		)
-		(property "Value" "74ACT139"
+		(property "Value" "74AC139"
 			(at 0 0 180)
 			(layer "F.SilkS")
@@
 	)
 	(segment
+		(start 106.3717 83.0037)
+		(end 106.68 83.312)
+		(width 0.35)
+		(layer "F.Cu")
+		(net 1)
+	)
+	(segment
 		(start 127.0429 60.3325)
 		(end 113.079 60.3325)
@@
 	(segment
 		(start 102.1645 88.2014)
-		(end 105.515 84.8509)
+		(end 102.9899 87.376)
 		(width 0.35)
 		(layer "F.Cu")
@@
 		(start 101.5891 88.7768)
 		(end 90.1033 88.7768)
+		(width 0.35)
+		(layer "F.Cu")
+		(net 1)
+	)
+	(segment
+		(start 104.902 85.598)
+		(end 104.902 85.4639)
+		(width 0.35)
+		(layer "F.Cu")
+		(net 1)
+	)
+	(segment
+		(start 104.7679 85.598)
+		(end 104.902 85.598)
 		(width 0.35)
 		(layer "F.Cu")
@@
 	)
 	(segment
+		(start 103.378 87.376)
+		(end 103.378 86.9879)
+		(width 0.35)
+		(layer "F.Cu")
+		(net 1)
+	)
+	(segment
 		(start 83.0284 59.4283)
 		(end 88.8743 59.4283)
@@
 	)
 	(segment
+		(start 102.9899 87.376)
+		(end 103.378 87.376)
+		(width 0.35)
+		(layer "F.Cu")
+		(net 1)
+	)
+	(segment
 		(start 91.4335 59.4245)
 		(end 90.152 60.706)
@@
 	)
 	(segment
-		(start 106.0755 83.2999)
-		(end 108.4329 80.9425)
-		(width 0.35)
-		(layer "F.Cu")
-		(net 1)
-	)
-	(segment
 		(start 128.778 76.962)
 		(end 129.4652 77.6492)
@@
 	)
 	(segment
+		(start 106.0755 83.2999)
+		(end 106.3717 83.0037)
+		(width 0.35)
+		(layer "F.Cu")
+		(net 1)
+	)
+	(segment
 		(start 108.4329 79.5109)
 		(end 108.925 79.0188)
@@
 		(start 81.28 60.125)
 		(end 82.3317 60.125)
+		(width 0.35)
+		(layer "F.Cu")
+		(net 1)
+	)
+	(segment
+		(start 106.68 83.312)
+		(end 106.68 84.836)
+		(width 0.35)
+		(layer "F.Cu")
+		(net 1)
+	)
+	(segment
+		(start 106.3717 83.0037)
+		(end 108.4329 80.9425)
 		(width 0.35)
 		(layer "F.Cu")
@@
 	)
 	(segment
+		(start 103.378 86.9879)
+		(end 104.7679 85.598)
+		(width 0.35)
+		(layer "F.Cu")
+		(net 1)
+	)
+	(segment
 		(start 85.598 93.726)
 		(end 85.09 93.726)
@@
 		(width 0.35)
 		(layer "F.Cu")
+		(net 1)
+	)
+	(segment
+		(start 104.902 85.4639)
+		(end 105.515 84.8509)
+		(width 0.35)
+		(layer "F.Cu")
+		(net 1)
+	)
+	(via
+		(at 106.68 84.836)
+		(size 0.6)
+		(drill 0.3)
+		(layers "F.Cu" "B.Cu")
 		(net 1)
 	)
@@
 	)
 	(via
+		(at 104.902 85.598)
+		(size 0.6)
+		(drill 0.3)
+		(layers "F.Cu" "B.Cu")
+		(net 1)
+	)
+	(via
 		(at 83.9228 72.5483)
 		(size 0.6)
@@
 		(size 0.6)
 		(drill 0.3)
+		(layers "F.Cu" "B.Cu")
+		(net 1)
+	)
+	(via
+		(at 103.378 87.376)
+		(size 0.6)
+		(drill 0.3)

Commit message: Add revision silkscreen
Other:
- board text added: "Rev. 0"
Changed lines of the file:
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@@
 		(layer "Edge.Cuts")
+	)
+	(gr_text "Rev. 0"
+		(at 124.841 60.706 0)
+		(layer "F.SilkS")
+		(effects
+			(font
+				(size 1 1)
+				(thickness 0.1)
+			)
+			(justify left bottom)
+		)
 	)
 	(gr_text "OtterX RAM\nEXPANSION"
